Commit message: axis 2 done

File: motion_cmd/urdf/azd3a_axis1_feedback.urdf.xacro (robot description, xacro)
@@ -15,5 +15,6 @@
     <!-- Conservative reference limits for the 30 mm actuator. No controller
          is loaded by the feedback-only launch. -->
-    <limit lower="0.000" upper="0.029" velocity="0.001" effort="40.0"/>
+    <!-- Manufacturer envelope; the runtime commissioning guard is tighter. -->
+    <limit lower="0.000" upper="0.030" velocity="0.040" effort="40.0"/>
   </joint>
   <ros2_control name="AZD3A_axis1_feedback" type="system">
@@ -21,5 +22,6 @@
       <plugin>ethercat_driver/EthercatDriver</plugin>
       <param name="master_id">0</param>
-      <param name="control_frequency">100</param>
+      <!-- AZD3A DC mode supports 0.5 ms or 1-8 ms; 200 Hz = 5 ms. -->
+      <param name="control_frequency">200</param>
       <param name="number_of_physical_drives">1</param>
     </hardware>
@@ -27,5 +29,5 @@
       <command_interface name="position">
         <param name="min">0.000</param>
-        <param name="max">0.029</param>
+        <param name="max">0.005</param>
       </command_interface>
       <state_interface name="position"/>

File: motion_cmd/urdf/azd3a_axis1_tiny_move.urdf.xacro (robot description, xacro)
@@ -12,5 +12,6 @@
     <child link="axis1_table"/>
     <axis xyz="1 0 0"/>
-    <limit lower="0.000" upper="0.029" velocity="0.001" effort="40.0"/>
+    <!-- Manufacturer envelope; the runtime commissioning guard is tighter. -->
+    <limit lower="0.000" upper="0.030" velocity="0.040" effort="40.0"/>
   </joint>
   <ros2_control name="AZD3A_axis1_tiny_move" type="system">
@@ -18,5 +19,6 @@
       <plugin>ethercat_driver/EthercatDriver</plugin>
       <param name="master_id">0</param>
-      <param name="control_frequency">100</param>
+      <!-- AZD3A DC mode supports 0.5 ms or 1-8 ms; 200 Hz = 5 ms. -->
+      <param name="control_frequency">200</param>
       <param name="number_of_physical_drives">1</param>
     </hardware>
@@ -24,5 +26,5 @@
       <command_interface name="position">
         <param name="min">0.000</param>
-        <param name="max">0.029</param>
+        <param name="max">0.015</param>
       </command_interface>
       <state_interface name="position"/>
@@ -31,4 +33,6 @@
         <param name="alias">0</param>
         <param name="position">0</param>
+        <!-- Hold measured position until the raw controller synchronizes. -->
+        <param name="position_startup_tolerance">0.00001</param>
         <param name="mode_of_operation">8</param>
         <param name="slave_config">$(find motor_controller)/config/azd3a_ked_cia402_slave.yaml</param>

Commit message: motor 1 2 4 6 done

File: motion_cmd/urdf/azd3a_axis1_feedback.urdf.xacro (robot description, xacro)
@@ -13,8 +13,6 @@
     <child link="axis1_table"/>
     <axis xyz="1 0 0"/>
-    <!-- Conservative reference limits for the 30 mm actuator. No controller
-         is loaded by the feedback-only launch. -->
-    <!-- Manufacturer envelope; the runtime commissioning guard is tighter. -->
-    <limit lower="0.000" upper="0.030" velocity="0.040" effort="40.0"/>
+    <!-- EZSM3LD040AZAK envelope. No controller is loaded by this launch. -->
+    <limit lower="0.000" upper="0.400" velocity="0.600" effort="43.0"/>
   </joint>
   <ros2_control name="AZD3A_axis1_feedback" type="system">
@@ -28,5 +26,5 @@
     <joint name="axis1_joint">
       <command_interface name="position">
-        <param name="min">0.000</param>
+        <param name="min">0.0000996</param>
         <param name="max">0.005</param>
       </command_interface>

File: motion_cmd/urdf/azd3a_axis1_tiny_move.urdf.xacro (robot description, xacro)
@@ -12,6 +12,6 @@
     <child link="axis1_table"/>
     <axis xyz="1 0 0"/>
-    <!-- Manufacturer envelope; the runtime commissioning guard is tighter. -->
-    <limit lower="0.000" upper="0.030" velocity="0.040" effort="40.0"/>
+    <!-- EZSM3LD040AZAK envelope; the runtime commissioning guard is tighter. -->
+    <limit lower="0.000" upper="0.400" velocity="0.600" effort="43.0"/>
   </joint>
   <ros2_control name="AZD3A_axis1_tiny_move" type="system">
@@ -25,6 +25,7 @@
     <joint name="axis1_joint">
       <command_interface name="position">
-        <param name="min">0.000</param>
-        <param name="max">0.015</param>
+        <!-- Keep 0.0996 mm clearance from provisional lower-end zero. -->
+        <param name="min">0.0000996</param>
+        <param name="max">0.005</param>
       </command_interface>
       <state_interface name="position"/>

Commit message: all motor implemented

File: motion_cmd/urdf/azd3a_axis1_feedback.urdf.xacro (robot description, xacro)
@@ -27,5 +27,5 @@
       <command_interface name="position">
         <param name="min">0.0000996</param>
-        <param name="max">0.005</param>
+        <param name="max">0.200</param>
       </command_interface>
       <state_interface name="position"/>

File: motion_cmd/urdf/azd3a_axis1_tiny_move.urdf.xacro (robot description, xacro)
@@ -27,5 +27,5 @@
         <!-- Keep 0.0996 mm clearance from provisional lower-end zero. -->
         <param name="min">0.0000996</param>
-        <param name="max">0.005</param>
+        <param name="max">0.200</param>
       </command_interface>
       <state_interface name="position"/>

File: motion_cmd/urdf/azd3a_motor1_motor2.urdf.xacro (robot description, xacro)
@@ -5,7 +5,8 @@
   <link name="motor4_table"/>
   <!--
-    One composite ros2_control joint represents two internal axes of the same
-    physical AZD3A slave: position is Motor 1; velocity is Motor 2. This keeps
-    one EtherCAT slave instance and two separately claimed command interfaces.
+    One composite ros2_control joint represents three internal axes of the same
+    physical AZD3A slave: position is Motor 1, velocity is Motor 2, and the
+    custom motor3_position interface is Motor 3. This keeps one EtherCAT slave
+    instance while allowing each axis to be claimed by a separate controller.
   -->
   <joint name="motor1_motor2" type="prismatic">
@@ -13,5 +14,5 @@
     <child link="motor1_table"/>
     <axis xyz="0 0 1"/>
-    <limit lower="0.0000996" upper="0.005" velocity="0.002" effort="43.0"/>
+    <limit lower="0.0000996" upper="0.200" velocity="0.015" effort="43.0"/>
   </joint>
   <joint name="motor4_joint" type="prismatic">
@@ -20,5 +21,5 @@
     <axis xyz="1 0 0"/>
     <!-- Tiny negative margin accepts the retained ABZO origin (-0.0034 mm). -->
-    <limit lower="-0.00001" upper="0.030" velocity="0.040" effort="10.0"/>
+    <limit lower="-0.00001" upper="0.030" velocity="0.008" effort="10.0"/>
   </joint>
   <ros2_control name="AZD3A_motor1_motor2" type="system">
@@ -32,5 +33,5 @@
       <command_interface name="position">
         <param name="min">0.0000996</param>
-        <param name="max">0.005</param>
+        <param name="max">0.200</param>
       </command_interface>
       <command_interface name="velocity">
@@ -38,6 +39,11 @@
         <param name="max">26.179938779914945</param>
       </command_interface>
+      <command_interface name="motor3_position">
+        <param name="min">0.0</param>
+        <param name="max">0.015</param>
+      </command_interface>
       <state_interface name="position"/>
       <state_interface name="velocity"/>
+      <state_interface name="motor3_position"/>
       <ec_module name="azd3a_motor1_motor2">
         <plugin>ethercat_generic_plugins/EcCiA402Drive</plugin>
@@ -48,4 +54,6 @@
         <param name="secondary_cia402_object_index_offset">0x0800</param>
         <param name="secondary_mode_of_operation">9</param>
+        <param name="tertiary_cia402_object_index_offset">0x1000</param>
+        <param name="tertiary_mode_of_operation">8</param>
         <param name="slave_config">$(find motor_controller)/config/azd3a_motor1_motor2_slave.yaml</param>
       </ec_module>
@@ -58,10 +66,12 @@
       </command_interface>
       <command_interface name="velocity">
-        <!-- Motor 6 conveyor: guarded to +/-5 output rpm. -->
-        <param name="min">-0.5235987755982988</param>
-        <param name="max">0.5235987755982988</param>
+        <!-- Motor 6 conveyor: guarded to +/-50 output rpm. -->
+        <param name="min">-5.235987755982989</param>
+        <param name="max">5.235987755982989</param>
       </command_interface>
+      <command_interface name="motor5_position"/>
       <state_interface name="position"/>
       <state_interface name="velocity"/>
+      <state_interface name="motor5_position"/>
       <ec_module name="azd3a_slave1_axis1_motor4">
         <plugin>ethercat_generic_plugins/EcCiA402Drive</plugin>
@@ -78,4 +88,6 @@
         <param name="secondary_cia402_object_index_offset">0x1000</param>
         <param name="secondary_mode_of_operation">9</param>
+        <param name="tertiary_cia402_object_index_offset">0x0800</param>
+        <param name="tertiary_mode_of_operation">8</param>
         <param name="slave_config">$(find motor_controller)/config/azd3a_motor4_motor6_slave.yaml</param>
       </ec_module>

File: motion_cmd/urdf/azd3a_motor5_commissioning.urdf.xacro (robot description, xacro)
@@ -1,25 +1,25 @@
 <?xml version="1.0"?>
-<robot xmlns:xacro="http://www.ros.org/wiki/xacro" name="azd3a_motor4_commissioning">
-  <link name="motor4_base"/>
-  <link name="motor4_table"/>
+<robot xmlns:xacro="http://www.ros.org/wiki/xacro" name="azd3a_motor5_commissioning">
+  <link name="motor5_base"/>
+  <link name="motor5_output"/>
   <link name="slave0_keepalive_base"/>
-  <link name="slave0_keepalive_table"/>
+  <link name="slave0_keepalive_output"/>
   <joint name="slave0_keepalive_mount" type="fixed">
-    <parent link="motor4_base"/>
+    <parent link="motor5_base"/>
     <child link="slave0_keepalive_base"/>
   </joint>
   <joint name="slave0_keepalive_joint" type="prismatic">
     <parent link="slave0_keepalive_base"/>
-    <child link="slave0_keepalive_table"/>
+    <child link="slave0_keepalive_output"/>
     <axis xyz="1 0 0"/>
     <limit lower="-1.0" upper="1.0" velocity="1.0" effort="1.0"/>
   </joint>
-  <joint name="motor4_joint" type="prismatic">
-    <parent link="motor4_base"/>
-    <child link="motor4_table"/>
-    <axis xyz="1 0 0"/>
-    <limit lower="-0.030" upper="0.030" velocity="0.008" effort="10.0"/>
+  <joint name="motor5_joint" type="continuous">
+    <parent link="motor5_base"/>
+    <child link="motor5_output"/>
+    <axis xyz="0 0 1"/>
+    <limit velocity="2.0943951023931953" effort="0.7"/>
   </joint>
-  <ros2_control name="AZD3A_motor4_commissioning" type="system">
+  <ros2_control name="AZD3A_motor5_commissioning" type="system">
     <hardware>
       <plugin>ethercat_driver/EthercatDriver</plugin>
@@ -28,9 +28,4 @@
       <param name="number_of_physical_drives">2</param>
     </hardware>
-    <!--
-      Slave 0 must receive cyclic outputs while slave 1 is controlled. This
-      GenericEcSlave sends only safe zero defaults and performs no CiA 402
-      state transitions, so Motors 1/2 cannot be enabled by this launch.
-    -->
     <joint name="slave0_keepalive_joint">
       <state_interface name="position"/>
@@ -42,15 +37,17 @@
       </ec_module>
     </joint>
-    <joint name="motor4_joint">
+    <joint name="motor5_joint">
       <command_interface name="position"/>
       <state_interface name="position"/>
-      <ec_module name="azd3a_slave1_axis1_motor4">
+      <state_interface name="velocity"/>
+      <ec_module name="azd3a_slave1_axis2_motor5">
         <plugin>ethercat_generic_plugins/EcCiA402Drive</plugin>
         <param name="alias">0</param>
         <param name="position">1</param>
-        <!-- One encoder count: reject any startup jump beyond 0.0001 mm. -->
-        <param name="position_startup_tolerance">0.0000001</param>
+        <param name="cia402_object_index_offset">0x0800</param>
+        <!-- Approximately one encoder count at 200,000 counts/revolution. -->
+        <param name="position_startup_tolerance">0.000032</param>
         <param name="mode_of_operation">8</param>
-        <param name="slave_config">$(find motor_controller)/config/azd3a_motor4_commissioning_slave.yaml</param>
+        <param name="slave_config">$(find motor_controller)/config/azd3a_motor5_commissioning_slave.yaml</param>
       </ec_module>
     </joint>

File: motion_cmd/urdf/azd3a_motor6_conveyor.urdf.xacro (robot description, xacro)
@@ -35,7 +35,7 @@
     <joint name="motor6_joint">
       <command_interface name="velocity">
-        <!-- Guarded commissioning launch is limited to +/-5 rpm. -->
-        <param name="min">-0.5235987755982988</param>
-        <param name="max">0.5235987755982988</param>
+        <!-- Guarded commissioning launch is limited to +/-50 rpm. -->
+        <param name="min">-5.235987755982989</param>
+        <param name="max">5.235987755982989</param>
       </command_interface>
       <state_interface name="position"/>
