Commit message: workspace and gui updated

File: motion_cmd/urdf/azd3a_motor1_motor2.urdf.xacro (robot description, xacro)
@@ -14,5 +14,5 @@
     <child link="motor1_table"/>
     <axis xyz="0 0 1"/>
-    <limit lower="0.0000996" upper="0.200" velocity="0.015" effort="43.0"/>
+    <limit lower="0.0" upper="0.400" velocity="0.015" effort="43.0"/>
   </joint>
   <joint name="motor4_joint" type="prismatic">
@@ -32,6 +32,6 @@
     <joint name="motor1_motor2">
       <command_interface name="position">
-        <param name="min">0.0000996</param>
-        <param name="max">0.200</param>
+        <param name="min">0.0</param>
+        <param name="max">0.400</param>
       </command_interface>
       <command_interface name="velocity">
@@ -41,9 +41,12 @@
       <command_interface name="motor3_position">
         <param name="min">0.0</param>
-        <param name="max">0.015</param>
+        <param name="max">0.020</param>
       </command_interface>
       <state_interface name="position"/>
       <state_interface name="velocity"/>
       <state_interface name="motor3_position"/>
+      <state_interface name="motor1_status"/>
+      <state_interface name="motor2_status"/>
+      <state_interface name="motor3_status"/>
       <ec_module name="azd3a_motor1_motor2">
         <plugin>ethercat_generic_plugins/EcCiA402Drive</plugin>
@@ -61,7 +64,7 @@
     <joint name="motor4_joint">
       <command_interface name="position">
-        <!-- GUI/guard commands remain 0..15 mm; this is startup margin only. -->
+        <!-- GUI/guard commands remain 0..20 mm; this is startup margin only. -->
         <param name="min">-0.00001</param>
-        <param name="max">0.015</param>
+        <param name="max">0.020</param>
       </command_interface>
       <command_interface name="velocity">
@@ -74,4 +77,8 @@
       <state_interface name="velocity"/>
       <state_interface name="motor5_position"/>
+      <state_interface name="motor6_position"/>
+      <state_interface name="motor4_status"/>
+      <state_interface name="motor5_status"/>
+      <state_interface name="motor6_status"/>
       <ec_module name="azd3a_slave1_axis1_motor4">
         <plugin>ethercat_generic_plugins/EcCiA402Drive</plugin>
