Commit message: 80% speed update

File: motion_cmd/urdf/azd3a_axis1_tiny_move.urdf.xacro (robot description, xacro)
@@ -27,5 +27,5 @@
         <!-- Keep 0.0996 mm clearance from provisional lower-end zero. -->
         <param name="min">0.0000996</param>
-        <param name="max">0.200</param>
+        <param name="max">0.400</param>
       </command_interface>
       <state_interface name="position"/>

File: motion_cmd/urdf/azd3a_axis2_tiny_spin.urdf.xacro (robot description, xacro)
@@ -7,5 +7,5 @@
     <child link="axis2_output"/>
     <axis xyz="0 0 1"/>
-    <!-- Official output maximum is 416 rpm; current machine requirement is <=250 rpm. -->
+    <!-- 80% of the official 416 rpm output maximum: 332.8 rpm. -->
     <limit velocity="43.563418" effort="0.7"/>
   </joint>
@@ -18,8 +18,8 @@
     </hardware>
     <joint name="axis2_joint">
-      <!-- +/-26.17993878 rad/s = +/-250 rpm machine requirement boundary. -->
+      <!-- +/-34.85073450 rad/s = +/-332.8 rpm (80% operating ceiling). -->
       <command_interface name="velocity">
-        <param name="min">-26.179938779914945</param>
-        <param name="max">26.179938779914945</param>
+        <param name="min">-34.85073450382277</param>
+        <param name="max">34.85073450382277</param>
       </command_interface>
       <state_interface name="position"/>

File: motion_cmd/urdf/azd3a_motor1_motor2.urdf.xacro (robot description, xacro)
@@ -14,5 +14,5 @@
     <child link="motor1_table"/>
     <axis xyz="0 0 1"/>
-    <limit lower="0.0" upper="0.400" velocity="0.015" effort="43.0"/>
+    <limit lower="0.0" upper="0.400" velocity="0.480" effort="43.0"/>
   </joint>
   <joint name="motor4_joint" type="prismatic">
@@ -21,5 +21,5 @@
     <axis xyz="1 0 0"/>
     <!-- Tiny negative margin accepts the retained ABZO origin (-0.0034 mm). -->
-    <limit lower="-0.00001" upper="0.030" velocity="0.008" effort="10.0"/>
+    <limit lower="-0.00001" upper="0.030" velocity="0.032" effort="10.0"/>
   </joint>
   <ros2_control name="AZD3A_motor1_motor2" type="system">
@@ -36,6 +36,6 @@
       </command_interface>
       <command_interface name="velocity">
-        <param name="min">-26.179938779914945</param>
-        <param name="max">26.179938779914945</param>
+        <param name="min">-34.85073450382277</param>
+        <param name="max">34.85073450382277</param>
       </command_interface>
       <command_interface name="motor3_position">
@@ -69,7 +69,7 @@
       </command_interface>
       <command_interface name="velocity">
-        <!-- Motor 6 conveyor: guarded to +/-50 output rpm. -->
-        <param name="min">-5.235987755982989</param>
-        <param name="max">5.235987755982989</param>
+        <!-- Motor 6 conveyor: 80% of the 60 rpm output maximum. -->
+        <param name="min">-5.026548245743669</param>
+        <param name="max">5.026548245743669</param>
       </command_interface>
       <command_interface name="motor5_position"/>

File: motion_cmd/urdf/azd3a_motor3_commissioning.urdf.xacro (robot description, xacro)
@@ -8,5 +8,5 @@
     <child link="motor3_table"/>
     <axis xyz="1 0 0"/>
-    <limit lower="-0.030" upper="0.030" velocity="0.008" effort="10.0"/>
+    <limit lower="-0.030" upper="0.030" velocity="0.032" effort="10.0"/>
   </joint>
   <joint name="slave1_keepalive_joint" type="prismatic">

File: motion_cmd/urdf/azd3a_motor4_commissioning.urdf.xacro (robot description, xacro)
@@ -19,5 +19,5 @@
     <child link="motor4_table"/>
     <axis xyz="1 0 0"/>
-    <limit lower="-0.030" upper="0.030" velocity="0.008" effort="10.0"/>
+    <limit lower="-0.030" upper="0.030" velocity="0.032" effort="10.0"/>
   </joint>
   <ros2_control name="AZD3A_motor4_commissioning" type="system">

File: motion_cmd/urdf/azd3a_motor6_conveyor.urdf.xacro (robot description, xacro)
@@ -35,7 +35,7 @@
     <joint name="motor6_joint">
       <command_interface name="velocity">
-        <!-- Guarded commissioning launch is limited to +/-50 rpm. -->
-        <param name="min">-5.235987755982989</param>
-        <param name="max">5.235987755982989</param>
+        <!-- 80% of 60 rpm permissible gearbox-output speed: +/-48 rpm. -->
+        <param name="min">-5.026548245743669</param>
+        <param name="max">5.026548245743669</param>
       </command_interface>
       <state_interface name="position"/>
